File: Hardware/IMU.kicad_sch (KiCad schematic)
At the start: 0 parts

Commit message: Developing HW
Parts:
- added C25: 2.2nF, Capacitor_SMD:C_0603_1608Metric, symbol Device:C_Small
- added C26, C27: 100nF, Capacitor_SMD:C_0603_1608Metric, symbol Device:C_Small
- added U7: MPU-6000, Sensor_Motion:InvenSense_QFN-24_4x4mm_P0.5mm, symbol Sensor_Motion:MPU-6000
Connections:
- new net: C26.1, U7.10 (REGOUT)
- new net: C25.1, U7.20 (CPOUT)
- new net GND: C25.2, C26.2, C27.2, U7.1 (CLKIN), U7.11 (FSYNC), U7.18 (GND)
- new net IMU_INT: U7.12 (INT)
- new net SPI_MISO: U7.9 (AD0/MISO)
- new net SPI_MOSI: U7.24 (SDA/MOSI)
- new net SPI_SCK: U7.23 (SCL/SCLK)
- new net SPI_SS0: U7.8 (~{CS})
- new net VCC: C27.1, U7.13 (VDD)
- no-connect marks 0 -> 2

Commit message: Developing HW
Parts:
- added R16: 51k, Resistor_SMD:R_0603_1608Metric, symbol Device:R_Small
- added R17: 0R, Resistor_SMD:R_0603_1608Metric, symbol Device:R_Small
- renumbered C27 to C25, C25 to C27, U7 to U6
Connections:
- net IMU_INT: now also R17.2; no longer U6.12 (INT)
- net VCC: now also R16.2
- net SPI_MISO renamed SPI1_MISO
- net SPI_MOSI renamed SPI1_MOSI
- net SPI_SCK renamed SPI1_SCK
- net SPI_SS0 renamed SPI1_NSS
- net SPI1_NSS: now also R16.1
- new net: R17.1, U6.12 (INT)

Commit message: Working on power source
Parts:
- C25, C26, C27: footprint Capacitor_SMD:C_0603_1608Metric -> Capacitor_SMD:C_0402_1005Metric
- R16, R17: footprint Resistor_SMD:R_0603_1608Metric -> Resistor_SMD:R_0402_1005Metric
Changed lines of the file:
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@@
 			)
 		)
-		(property "Footprint" "Resistor_SMD:R_0603_1608Metric"
+		(property "Footprint" "Resistor_SMD:R_0402_1005Metric"
 			(at 160.02 78.74 0)
 			(effects
@@
 			)
 		)
-		(property "Footprint" "Capacitor_SMD:C_0603_1608Metric"
+		(property "Footprint" "Capacitor_SMD:C_0402_1005Metric"
 			(at 161.29 97.79 0)
 			(effects
@@
 			)
 		)
-		(property "Footprint" "Capacitor_SMD:C_0603_1608Metric"
+		(property "Footprint" "Capacitor_SMD:C_0402_1005Metric"
 			(at 166.37 97.79 0)
 			(effects
@@
 			)
 		)
-		(property "Footprint" "Resistor_SMD:R_0603_1608Metric"
+		(property "Footprint" "Resistor_SMD:R_0402_1005Metric"
 			(at 90.17 64.77 0)
 			(effects
@@
 			)
 		)
-		(property "Footprint" "Capacitor_SMD:C_0603_1608Metric"
+		(property "Footprint" "Capacitor_SMD:C_0402_1005Metric"
 			(at 133.35 62.23 0)
 			(effects
