File: Hardware/LEDs_Buzzer.kicad_sch (KiCad schematic)
At the start: 36 parts, among them Q1 BC848, Q2 BC848, Q3 BC848, U2 TCA9534

Commit message: Developing HW
Changed lines of the file:
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@@
 	(text_box "I_{B} = I_{C}/β = 95/180 = 0.53 mA\n\nR_{B} = (V_{in} - V_{BE})/I_{B} = (3.3 - 0.7)/0.53 = 4.9 kΩ\n\n\nObs: (BC848) I_{C_max} = 100 mA"
 		(exclude_from_sim yes)
-		(at 62.23 171.45 0)
+		(at 62.23 173.99 0)
 		(size 44.45 11.43)
 		(stroke

Commit message: Developing HW
Parts:
- BZ1: footprint (none) -> Buzzer_Beeper:PUIAudio_SMT_0825_S_4_R
- D10: renamed from D5; footprint (none) -> LED_SMD:LED_0603_1608Metric
- D11: renamed from D6; footprint (none) -> LED_SMD:LED_0603_1608Metric
- D12: renamed from D9; footprint (none) -> Diode_SMD:D_SOD-123
- D4: renamed from D7; footprint (none) -> LED_SMD:LED_0805_2012Metric
- D5: renamed from D8; footprint (none) -> LED_SMD:LED_0805_2012Metric
- D6: renamed from D1; footprint (none) -> LED_SMD:LED_0603_1608Metric
- D7: renamed from D2; footprint (none) -> LED_SMD:LED_0603_1608Metric
- D8: renamed from D3; footprint (none) -> LED_SMD:LED_0603_1608Metric
- D9: renamed from D4; footprint (none) -> LED_SMD:LED_0603_1608Metric
- JP10: renamed from JP7; footprint (none) -> Jumper:SolderJumper-2_P1.3mm_Open_RoundedPad1.0x1.5mm
- JP11: renamed from JP8; footprint (none) -> Jumper:SolderJumper-2_P1.3mm_Open_RoundedPad1.0x1.5mm
- JP6: renamed from JP3; footprint (none) -> Jumper:SolderJumper-2_P1.3mm_Open_RoundedPad1.0x1.5mm
- JP7: renamed from JP4; footprint (none) -> Jumper:SolderJumper-2_P1.3mm_Open_RoundedPad1.0x1.5mm
- JP8: renamed from JP5; footprint (none) -> Jumper:SolderJumper-2_P1.3mm_Open_RoundedPad1.0x1.5mm
- JP9: renamed from JP6; footprint (none) -> Jumper:SolderJumper-2_P1.3mm_Open_RoundedPad1.0x1.5mm
- R18: renamed from R14; footprint (none) -> Resistor_SMD:R_0603_1608Metric
- R19: renamed from R15; footprint (none) -> Resistor_SMD:R_0603_1608Metric
- R20: renamed from R17; footprint (none) -> Resistor_SMD:R_0603_1608Metric
- R21: renamed from R18; footprint (none) -> Resistor_SMD:R_0603_1608Metric
- R22: renamed from R4; footprint (none) -> Resistor_SMD:R_0603_1608Metric
- R23: renamed from R9; footprint (none) -> Resistor_SMD:R_0603_1608Metric
- R24: renamed from R10; footprint (none) -> Resistor_SMD:R_0603_1608Metric
- R25: renamed from R11; footprint (none) -> Resistor_SMD:R_0603_1608Metric
- R26: renamed from R12; footprint (none) -> Resistor_SMD:R_0603_1608Metric
- R27: renamed from R13; footprint (none) -> Resistor_SMD:R_0603_1608Metric
- R28: renamed from R16; footprint (none) -> Resistor_SMD:R_0603_1608Metric
- R29: renamed from R19; footprint (none) -> Resistor_SMD:R_0603_1608Metric
- R30: renamed from R20; footprint (none) -> Resistor_SMD:R_0603_1608Metric
- R31: renamed from R21; footprint (none) -> Resistor_SMD:R_0603_1608Metric
- U8: renamed from U2; footprint (none) -> Package_SO:SOIC-16W_7.5x10.3mm_P1.27mm
- renumbered C15 to C30, C14 to C31, Q1 to Q5, Q2 to Q6, Q3 to Q7
Connections:
- net IO_P1: now reaches JP10.2 (B)
- net IO_P1: now also U8.5 (P1); no longer U8.7 (P3)
- net IO_P0: now reaches JP11.2 (B)
- net IO_P0: now also U8.4 (P0); no longer U8.6 (P2)
- net IO_P2: now reaches R21.1
- net IO_P2: now also U8.6 (P2); no longer U8.4 (P0)
- net IO_P6: now reaches JP7.2 (B), U8.11 (P6)
- net IO_P3: now reaches R20.1
- net IO_P3: now also U8.7 (P3); no longer U8.5 (P1)
- net IO_P7: now reaches JP6.2 (B), U8.12 (P7)
- net IO_P5: now reaches JP8.2 (B), U8.10 (P5)
- net IO_P4: now reaches JP9.2 (B), U8.9 (P4)
- no-connect marks 1 -> 5

Commit message: Developing HW - routing
Parts:
- JP10, JP11, JP6, JP7, JP8, JP9: footprint Jumper:SolderJumper-2_P1.3mm_Open_RoundedPad1.0x1.5mm -> BRS_Footprints:SMD_SolderJumper_Small
- U8: footprint Package_SO:SOIC-16W_7.5x10.3mm_P1.27mm -> Package_SO:TSSOP-16_4.4x5mm_P0.65mm
Changed lines of the file:
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@@
 			)
 		)
-		(property "Footprint" "Jumper:SolderJumper-2_P1.3mm_Open_RoundedPad1.0x1.5mm"
+		(property "Footprint" "BRS_Footprints:SMD_SolderJumper_Small"
 			(at 140.97 81.28 0)
 			(effects
@@
 			)
 		)
-		(property "Footprint" "Jumper:SolderJumper-2_P1.3mm_Open_RoundedPad1.0x1.5mm"
+		(property "Footprint" "BRS_Footprints:SMD_SolderJumper_Small"
 			(at 153.67 81.28 0)
 			(effects
@@
 			)
 		)
-		(property "Footprint" "Jumper:SolderJumper-2_P1.3mm_Open_RoundedPad1.0x1.5mm"
+		(property "Footprint" "BRS_Footprints:SMD_SolderJumper_Small"
 			(at 102.87 81.28 0)
 			(effects
@@
 			)
 		)
-		(property "Footprint" "Jumper:SolderJumper-2_P1.3mm_Open_RoundedPad1.0x1.5mm"
+		(property "Footprint" "BRS_Footprints:SMD_SolderJumper_Small"
 			(at 90.17 81.28 0)
 			(effects
@@
 			)
 		)
-		(property "Footprint" "Jumper:SolderJumper-2_P1.3mm_Open_RoundedPad1.0x1.5mm"
+		(property "Footprint" "BRS_Footprints:SMD_SolderJumper_Small"
 			(at 115.57 81.28 0)
 			(effects
@@
 			)
 		)
-		(property "Footprint" "Jumper:SolderJumper-2_P1.3mm_Open_RoundedPad1.0x1.5mm"
+		(property "Footprint" "BRS_Footprints:SMD_SolderJumper_Small"
 			(at 128.27 81.28 0)
 			(effects
@@
 			)
 		)
-		(property "Footprint" "Package_SO:SOIC-16W_7.5x10.3mm_P1.27mm"
+		(property "Footprint" "Package_SO:TSSOP-16_4.4x5mm_P0.65mm"
 			(at 97.79 71.12 0)
 			(effects

Commit message: Working on power source
Parts:
- C30, C31: footprint Capacitor_SMD:C_0603_1608Metric -> Capacitor_SMD:C_0402_1005Metric
- JP10, JP11, JP6, JP7, JP8, JP9: footprint BRS_Footprints:SMD_SolderJumper_Small -> BRS_Footprints:SMD_SolderJumper_Micro
- R18, R19, R20, R21, R22, R23, R24, R25, R26, R27, R28, R29, R30, R31: footprint Resistor_SMD:R_0603_1608Metric -> Resistor_SMD:R_0402_1005Metric
Changed lines of the file:
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@@
 			)
 		)
-		(property "Footprint" "Resistor_SMD:R_0603_1608Metric"
+		(property "Footprint" "Resistor_SMD:R_0402_1005Metric"
 			(at 215.9 74.93 0)
 			(effects
@@
 			)
 		)
-		(property "Footprint" "Resistor_SMD:R_0603_1608Metric"
+		(property "Footprint" "Resistor_SMD:R_0402_1005Metric"
 			(at 102.87 87.63 0)
 			(effects
@@
 			)
 		)
-		(property "Footprint" "Resistor_SMD:R_0603_1608Metric"
+		(property "Footprint" "Resistor_SMD:R_0402_1005Metric"
 			(at 173.99 93.98 0)
 			(effects
@@
 			)
 		)
-		(property "Footprint" "BRS_Footprints:SMD_SolderJumper_Small"
+		(property "Footprint" "BRS_Footprints:SMD_SolderJumper_Micro"
 			(at 140.97 81.28 0)
 			(effects
@@
 			)
 		)
-		(property "Footprint" "Resistor_SMD:R_0603_1608Metric"
+		(property "Footprint" "Resistor_SMD:R_0402_1005Metric"
 			(at 153.67 87.63 0)
 			(effects
@@
 			)
 		)
-		(property "Footprint" "Resistor_SMD:R_0603_1608Metric"
+		(property "Footprint" "Resistor_SMD:R_0402_1005Metric"
 			(at 182.88 74.93 0)
 			(effects
@@
 			)
 		)
-		(property "Footprint" "Resistor_SMD:R_0603_1608Metric"
+		(property "Footprint" "Resistor_SMD:R_0402_1005Metric"
 			(at 115.57 87.63 0)
 			(effects
@@
 			)
 		)
-		(property "Footprint" "BRS_Footprints:SMD_SolderJumper_Small"
+		(property "Footprint" "BRS_Footprints:SMD_SolderJumper_Micro"
 			(at 153.67 81.28 0)
 			(effects
@@
 			)
 		)
-		(property "Footprint" "Resistor_SMD:R_0603_1608Metric"
+		(property "Footprint" "Resistor_SMD:R_0402_1005Metric"
 			(at 128.27 87.63 0)
 			(effects
@@
 			)
 		)
-		(property "Footprint" "Resistor_SMD:R_0603_1608Metric"
+		(property "Footprint" "Resistor_SMD:R_0402_1005Metric"
 			(at 207.01 86.36 0)
 			(effects
@@
 			)
 		)
-		(property "Footprint" "Resistor_SMD:R_0603_1608Metric"
+		(property "Footprint" "Resistor_SMD:R_0402_1005Metric"
 			(at 82.55 160.02 0)
 			(effects
@@
 			)
 		)
-		(property "Footprint" "Capacitor_SMD:C_0603_1608Metric"
+		(property "Footprint" "Capacitor_SMD:C_0402_1005Metric"
 			(at 63.5 34.29 0)
 			(effects
@@
 			)
 		)
-		(property "Footprint" "BRS_Footprints:SMD_SolderJumper_Small"
+		(property "Footprint" "BRS_Footprints:SMD_SolderJumper_Micro"
 			(at 102.87 81.28 0)
 			(effects
@@
 			)
 		)
-		(property "Footprint" "Resistor_SMD:R_0603_1608Metric"
+		(property "Footprint" "Resistor_SMD:R_0402_1005Metric"
 			(at 173.99 86.36 0)
 			(effects
@@
 			)
 		)
-		(property "Footprint" "Resistor_SMD:R_0603_1608Metric"
+		(property "Footprint" "Resistor_SMD:R_0402_1005Metric"
 			(at 90.17 87.63 0)
 			(effects
@@
 			)
 		)
-		(property "Footprint" "Capacitor_SMD:C_0603_1608Metric"
+		(property "Footprint" "Capacitor_SMD:C_0402_1005Metric"
 			(at 53.34 34.29 0)
 			(effects
@@
 			)
 		)
-		(property "Footprint" "Resistor_SMD:R_0603_1608Metric"
+		(property "Footprint" "Resistor_SMD:R_0402_1005Metric"
 			(at 140.97 87.63 0)
 			(effects
@@
 			)
 		)
-		(property "Footprint" "BRS_Footprints:SMD_SolderJumper_Small"
+		(property "Footprint" "BRS_Footprints:SMD_SolderJumper_Micro"
 			(at 90.17 81.28 0)
 			(effects
@@
 			)
 		)
-		(property "Footprint" "Resistor_SMD:R_0603_1608Metric"
+		(property "Footprint" "Resistor_SMD:R_0402_1005Metric"
 			(at 77.47 154.94 0)
 			(effects
@@
 			)
 		)
-		(property "Footprint" "BRS_Footprints:SMD_SolderJumper_Small"
+		(property "Footprint" "BRS_Footprints:SMD_SolderJumper_Micro"
 			(at 115.57 81.28 0)
 			(effects
@@
 			)
 		)
-		(property "Footprint" "BRS_Footprints:SMD_SolderJumper_Small"
+		(property "Footprint" "BRS_Footprints:SMD_SolderJumper_Micro"
 			(at 128.27 81.28 0)
 			(effects
@@
 			)
 		)
-		(property "Footprint" "Resistor_SMD:R_0603_1608Metric"
+		(property "Footprint" "Resistor_SMD:R_0402_1005Metric"
 			(at 207.01 93.98 0)
 			(effects
