File: Hardware/MCU.kicad_sch (KiCad schematic)
At the start: 28 parts, among them J1 EXT_GPIOS, J3 SWD/ExtTrig, SW1 SW_MCU_NRST, U1 STM32F411CEUx, Y1 16MHz

Commit message: Developing HW
Parts:
- added C17: 10nF, Capacitor_SMD:C_0603_1608Metric, symbol Device:C_Small
- added R25: 620k, Resistor_SMD:R_0603_1608Metric, symbol Device:R_Small
- added R26: 220k, Resistor_SMD:R_0603_1608Metric, symbol Device:R_Small
Connections:
- net ADC_BAT: now also C17.1, R25.1, R26.2
- net GND: now also C17.2, R26.1
- net MAIN_PWR renamed BOARD_PWR
- new net +BATT: R25.2
Other:
- note added: "BATTERY ADC"
- moved on the sheet: C1, C10, C11, C12, C13, C2, C3, C4, C5, C6, C7, C8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

Commit message: Developing HW
Parts:
- added H1, H3, H5, H7: SupPCB, MountingHole:MountingHole_2.2mm_M2_DIN965, symbol Mechanical:MountingHole
- added H2, H4, H6: ToolingHole, TFG_Footprints:JLCPCB_Tooling_Hole, symbol Mechanical:MountingHole
- JP3: renamed from JP1; footprint (none) -> Jumper:SolderJumper-3_P1.3mm_Open_RoundedPad1.0x1.5mm
- JP4: renamed from JP2; footprint (none) -> Jumper:SolderJumper-3_P1.3mm_Open_RoundedPad1.0x1.5mm
- R7: renamed from R6; footprint Resistor_SMD:R_0603_1608Metric -> Resistor_SMD:R_0402_1005Metric
- R8: renamed from R7; footprint Resistor_SMD:R_0603_1608Metric -> Resistor_SMD:R_0402_1005Metric
- renumbered C12 to C10, C8 to C12, C10 to C13, C3 to C14, C7 to C15, C4 to C16, C13 to C17, C5 to C18, C17 to C19, C1 to C6, C2 to C7, C6 to C8, J1 to J4, R26 to R10, R3 to R2, R5 to R3, R1 to R4, R8 to R5, R2 to R6, R25 to R9, SW1 to SW2, U1 to U3
Connections:
- net EXT_A1 is gone; now on net EXT_B1: J4.3 (Pin_3)
- net EXT_A2 is gone; now on net UART1_TX: J4.4 (Pin_4)
- net EXT_A3 is gone; now on net UART1_RX: J4.5 (Pin_5)
- net EXT_C0 is gone; now on net EXT_A8: J4.1 (Pin_1)
- net EXT_C1 is gone; now on net EXT_B0: J4.2 (Pin_2)
- net BRS_RBF: now also U3.11 (PA1); no longer U3.26 (PB13)
- net BRS_RCV: now also U3.12 (PA2); no longer U3.27 (PB14)
- net EXT_B0: now reaches U3.18 (PB0)
- net EXT_B1: now reaches U3.19 (PB1)
- net SPI2_SCK: now reaches U3.21 (PB10)
- net SPI2_NSS1: now reaches U3.25 (PB12)
- net SPI2_MOSI: now reaches U3.28 (PB15)
- net EXT_A8: now reaches U3.29 (PA8)
- net I2C_INT: no longer names the net of U3.41 (PB5)
- net SPI_MISO renamed SPI1_MISO
- net SPI_MOSI renamed SPI1_MOSI
- net SPI_SCK renamed SPI1_SCK
- net SPI_SS0 renamed IMU_INT
- net SPI_SS1 renamed SPI1_NSS
- new net SPI2_MISO: U3.27 (PB14)
- new net SPI2_NSS0: U3.26 (PB13)
- no-connect marks 14 -> 7
Other:
- note added: "MOUNTING"

Commit message: Developing HW - routing
Parts:
- JP3, JP4: footprint Jumper:SolderJumper-3_P1.3mm_Open_RoundedPad1.0x1.5mm -> BRS_Footprints:SMD_SolderJumper_Triple_Small
Connections:
- net +BATT renamed HV_PWR_IN
Other:
- moved on the sheet: C19, R10, R9

Commit message: Working on power source
Parts:
- C11, C16, C17, C18, C19, C6: footprint Capacitor_SMD:C_0603_1608Metric -> Capacitor_SMD:C_0402_1005Metric
- JP3, JP4: footprint BRS_Footprints:SMD_SolderJumper_Triple_Small -> BRS_Footprints:SMD_SolderJumper_Triple_Micro
- R10, R2, R4, R5, R6, R9: footprint Resistor_SMD:R_0603_1608Metric -> Resistor_SMD:R_0402_1005Metric
Changed lines of the file:
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@@
 			)
 		)
-		(property "Footprint" "Resistor_SMD:R_0603_1608Metric"
+		(property "Footprint" "Resistor_SMD:R_0402_1005Metric"
 			(at 110.49 153.67 0)
 			(effects
@@
 			)
 		)
-		(property "Footprint" "Capacitor_SMD:C_0603_1608Metric"
+		(property "Footprint" "Capacitor_SMD:C_0402_1005Metric"
 			(at 105.41 158.75 0)
 			(effects
@@
 			)
 		)
-		(property "Footprint" "Resistor_SMD:R_0603_1608Metric"
+		(property "Footprint" "Resistor_SMD:R_0402_1005Metric"
 			(at 110.49 110.49 0)
 			(effects
@@
 			)
 		)
-		(property "Footprint" "Capacitor_SMD:C_0603_1608Metric"
+		(property "Footprint" "Capacitor_SMD:C_0402_1005Metric"
 			(at 104.14 54.61 0)
 			(effects
@@
 			)
 		)
-		(property "Footprint" "BRS_Footprints:SMD_SolderJumper_Triple_Small"
+		(property "Footprint" "BRS_Footprints:SMD_SolderJumper_Triple_Micro"
 			(at 125.73 153.67 0)
 			(effects
@@
 			)
 		)
-		(property "Footprint" "BRS_Footprints:SMD_SolderJumper_Triple_Small"
+		(property "Footprint" "BRS_Footprints:SMD_SolderJumper_Triple_Micro"
 			(at 176.53 153.67 0)
 			(effects
@@
 			)
 		)
-		(property "Footprint" "Resistor_SMD:R_0603_1608Metric"
+		(property "Footprint" "Resistor_SMD:R_0402_1005Metric"
 			(at 99.06 232.41 0)
 			(effects
@@
 			)
 		)
-		(property "Footprint" "Capacitor_SMD:C_0603_1608Metric"
+		(property "Footprint" "Capacitor_SMD:C_0402_1005Metric"
 			(at 110.49 120.65 0)
 			(effects
@@
 			)
 		)
-		(property "Footprint" "Capacitor_SMD:C_0603_1608Metric"
+		(property "Footprint" "Capacitor_SMD:C_0402_1005Metric"
 			(at 156.21 158.75 0)
 			(effects
@@
 			)
 		)
-		(property "Footprint" "Resistor_SMD:R_0603_1608Metric"
+		(property "Footprint" "Resistor_SMD:R_0402_1005Metric"
 			(at 99.06 224.79 0)
 			(effects
@@
 			)
 		)
-		(property "Footprint" "Capacitor_SMD:C_0603_1608Metric"
+		(property "Footprint" "Capacitor_SMD:C_0402_1005Metric"
 			(at 160.02 81.28 0)
 			(effects
@@
 			)
 		)
-		(property "Footprint" "Resistor_SMD:R_0603_1608Metric"
+		(property "Footprint" "Resistor_SMD:R_0402_1005Metric"
 			(at 161.29 153.67 0)
 			(effects
@@
 			)
 		)
-		(property "Footprint" "Resistor_SMD:R_0603_1608Metric"
+		(property "Footprint" "Resistor_SMD:R_0402_1005Metric"
 			(at 105.41 116.84 0)
 			(effects
@@
 			)
 		)
-		(property "Footprint" "Capacitor_SMD:C_0603_1608Metric"
+		(property "Footprint" "Capacitor_SMD:C_0402_1005Metric"
 			(at 104.14 232.41 0)
 			(effects
