File: Hardware/Power_Tree.kicad_sch (KiCad schematic)
At the start: 0 parts

Commit message: Developing HW
Parts:
- added C18, C19: TBD, symbol Device:C_Small
- added C20, C21: 100n, symbol Device:C_Small
- added C22: 10u, symbol Device:C_Small
- added D11, D12: TBD, symbol Device:D_Schottky_Small
- added D13: RED, symbol Device:LED_Small
- added J5: BATTERY, symbol Connector_Generic:Conn_02x02_Row_Letter_First
- added J6: USB_C_Receptacle_USB2.0_14P, symbol Connector:USB_C_Receptacle_USB2.0_14P
- added JP10: Jumper_2_Small_Open, symbol Jumper:Jumper_2_Small_Open
- added JP9: USB_PWR_JP, symbol Jumper:Jumper_2_Small_Open
- added Q5, Q6: PMOS, symbol Simulation_SPICE:PMOS
- added R27: 1k2, symbol Device:R_Small
- added SW2: ON/OFF MECH, symbol Switch:SW_DIP_x01
- added U4: AMS1117-3.3, Package_TO_SOT_SMD:SOT-223-3_TabPin2, symbol Regulator_Linear:AMS1117-3.3
- added U5: USBLC6-2, Package_TO_SOT_SMD:SOT-23-6, symbol Power_Protection:USBLC6-2SC6
Connections:
- new net: J6.A7 (D-), J6.B7 (D-), U5.1 (I/O1)
- new net: J6.A6 (D+), J6.B6 (D+), U5.3 (I/O2)
- new net: D11.1 (K), Q5.1 (D)
- new net: D13.2 (A), R27.2
- new net: JP10.1 (A), R27.1
- new net: D12.1 (K), JP9.1 (A)
- new net +BATT: JP9.2 (B), Q5.3 (S), SW2.1
- new net BAT+: D11.2 (A), J5.a1 (Pin_a1), J5.a2 (Pin_a2)
- new net BOARD_PWR: Q5.2 (G)
- new net GND: C18.2, C19.2, C20.2, C21.2, C22.2, D13.1 (K), J5.b1 (Pin_b1), J5.b2 (Pin_b2), J6.A1 (GND), J6.A12 (GND), J6.B1 (GND), J6.B12 (GND), U4.1 (GND), U5.2 (GND)
- new net HV_PWR_IN: C19.1, SW2.2, U4.3 (VI)
- new net SENS_PWR: Q6.2 (G)
- new net USB_DM: U5.6 (I/O1)
- new net USB_DP: U5.4 (I/O2)
- new net VBUS: C20.1, C21.1, C22.1, D12.2 (A), J6.A4 (VBUS), J6.A9 (VBUS), J6.B4 (VBUS), J6.B9 (VBUS), U5.5 (VBUS)
- new net VCC: Q6.3 (S)
- new net VDD: C18.1, JP10.2 (B), Q6.1 (D), U4.2 (VO)
- no-connect marks 0 -> 3
Other:
- note added: "This will not be the actual power supply. No LDOs will be used for final version!"

Commit message: Developing HW
Parts:
- added J8: GND, Connector_PinHeader_2.54mm:PinHeader_1x03_P2.54mm_Vertical, symbol Connector:Conn_01x03_Pin
- added J9: 3V3, Connector_PinHeader_2.54mm:PinHeader_1x03_P2.54mm_Vertical, symbol Connector:Conn_01x03_Pin
- added TP1: TestPoint_Small, TestPoint:TestPoint_Pad_D1.5mm, symbol Connector:TestPoint_Small
- C1: renamed from C19; footprint (none) -> Capacitor_SMD:C_0603_1608Metric
- C2: renamed from C18; footprint (none) -> Capacitor_SMD:C_0603_1608Metric
- C3: renamed from C22; footprint (none) -> Capacitor_SMD:C_0603_1608Metric
- C4: renamed from C21; footprint (none) -> Capacitor_SMD:C_0603_1608Metric
- C5: renamed from C20; footprint (none) -> Capacitor_SMD:C_0603_1608Metric
- D1: renamed from D11; footprint (none) -> Diode_SMD:D_SOD-123
- D2: renamed from D12; footprint (none) -> Diode_SMD:D_SOD-123
- D3: renamed from D13; footprint (none) -> LED_SMD:LED_0603_1608Metric
- J1: renamed from J5; footprint (none) -> Connector_Molex:Molex_Micro-Fit_3.0_43045-0412_2x02_P3.00mm_Vertical; symbol Connector_Generic:Conn_02x02_Row_Letter_First -> Connector_Generic:Conn_02x02_Odd_Even
- J2: renamed from J6; footprint (none) -> Connector_USB:USB_C_Receptacle_GCT_USB4105-xx-A_16P_TopMnt_Horizontal
- JP1: renamed from JP9; footprint (none) -> Jumper:SolderJumper-2_P1.3mm_Open_RoundedPad1.0x1.5mm
- JP2: renamed from JP10; footprint (none) -> Jumper:SolderJumper-2_P1.3mm_Open_RoundedPad1.0x1.5mm
- Q1: renamed from Q5; footprint (none) -> Package_TO_SOT_SMD:SOT-23
- Q2: renamed from Q6; footprint (none) -> Package_TO_SOT_SMD:SOT-23
- R1: renamed from R27; footprint (none) -> Resistor_SMD:R_0603_1608Metric
- SW1: renamed from SW2; footprint (none) -> Button_Switch_THT:SW_DIP_SPSTx03_Slide_6.7x9.18mm_W7.62mm_P2.54mm_LowProfile; symbol Switch:SW_DIP_x01 -> Switch:SW_DIP_x03
- renumbered U4 to U1, U5 to U2
Connections:
- net +BATT: now also SW1.2, SW1.3
- net BAT+: now also J1.1 (Pin_1), J1.3 (Pin_3); no longer J1.a1 (Pin_a1), J1.a2 (Pin_a2)
- net GND: now also J1.2 (Pin_2), J1.4 (Pin_4), J8.1 (Pin_1), J8.2 (Pin_2), J8.3 (Pin_3); no longer J1.b1 (Pin_b1), J1.b2 (Pin_b2)
- net HV_PWR_IN: now also SW1.4, SW1.5, SW1.6; no longer SW1.2
- net VDD: now also J9.1 (Pin_1), J9.2 (Pin_2), J9.3 (Pin_3)
- no-connect marks 3 -> 4

Commit message: Developing HW - routing
Parts:
- added J10: VCC, Connector_PinHeader_2.54mm:PinHeader_1x03_P2.54mm_Vertical, symbol Connector:Conn_01x03_Pin
- J9: value 3V3 -> VDD
- JP2: footprint Jumper:SolderJumper-2_P1.3mm_Open_RoundedPad1.0x1.5mm -> BRS_Footprints:SMD_SolderJumper_Small
Connections:
- net VCC: now also J10.1 (Pin_1), J10.2 (Pin_2), J10.3 (Pin_3)
Changed lines of the file:
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@@
 	)
 	(junction
+		(at 204.47 110.49)
+		(diameter 0)
+		(color 0 0 0 0)
+	)
+	(junction
 		(at 184.15 57.15)
 		(diameter 0)
@@
 	)
 	(junction
+		(at 204.47 107.95)
+		(diameter 0)
+		(color 0 0 0 0)
+	)
+	(junction
 		(at 119.38 43.18)
 		(diameter 0)
@@
 	(wire
 		(pts
+			(xy 204.47 107.95) (xy 204.47 110.49)
+		)
+		(stroke
+			(width 0)
+			(type default)
+		)
+	)
+	(wire
+		(pts
 			(xy 58.42 83.82) (xy 59.69 83.82)
 		)
@@
 	(wire
 		(pts
+			(xy 204.47 106.68) (xy 204.47 107.95)
+		)
+		(stroke
+			(width 0)
+			(type default)
+		)
+	)
+	(wire
+		(pts
 			(xy 60.96 41.91) (xy 59.69 41.91)
 		)
@@
 	(wire
 		(pts
+			(xy 204.47 110.49) (xy 204.47 113.03)
+		)
+		(stroke
+			(width 0)
+			(type default)
+		)
+	)
+	(wire
+		(pts
 			(xy 59.69 41.91) (xy 59.69 44.45)
 		)
@@
 	(wire
 		(pts
+			(xy 205.74 107.95) (xy 204.47 107.95)
+		)
+		(stroke
+			(width 0)
+			(type default)
+		)
+	)
+	(wire
+		(pts
 			(xy 185.42 90.17) (xy 184.15 90.17)
 		)
@@
 	(wire
 		(pts
+			(xy 205.74 110.49) (xy 204.47 110.49)
+		)
+		(stroke
+			(width 0)
+			(type default)
+		)
+	)
+	(wire
+		(pts
 			(xy 87.63 63.5) (xy 88.9 63.5)
 		)
@@
 	(wire
 		(pts
+			(xy 205.74 113.03) (xy 204.47 113.03)
+		)
+		(stroke
+			(width 0)
+			(type default)
+		)
+	)
+	(wire
+		(pts
 			(xy 82.55 93.98) (xy 81.28 93.98)
 		)
@@
 			)
 		)
-		(property "Footprint" "Jumper:SolderJumper-2_P1.3mm_Open_RoundedPad1.0x1.5mm"
+		(property "Footprint" "BRS_Footprints:SMD_SolderJumper_Small"
 			(at 217.17 67.31 0)
 			(effects
@@
 			)
 		)
-		(property "Value" "3V3"
+		(property "Value" "VDD"
 			(at 198.12 118.11 0)
 			(effects
@@
 	)
 	(symbol
+		(lib_id "Connector:Conn_01x03_Pin")
+		(at 210.82 110.49 0)
+		(mirror y)
+		(unit 1)
+		(exclude_from_sim no)
+		(in_bom no)
+		(on_board yes)
+		(dnp no)
+		(property "Reference" "J10"
+			(at 209.55 115.57 0)
+			(effects
+				(font
+					(size 1.27 1.27)
+				)
+			)
+		)
+		(property "Value" "VCC"
+			(at 209.55 118.11 0)
+			(effects
+				(font
+					(size 1.27 1.27)
+				)
+			)
+		)
+		(property "Footprint" "Connector_PinHeader_2.54mm:PinHeader_1x03_P2.54mm_Vertical"
+			(at 210.82 110.49 0)
+			(effects
+				(font
+					(size 1.27 1.27)
+				)
+				(hide yes)
+			)
+		)
+		(property "Datasheet" "~"
+			(at 210.82 110.49 0)
+			(effects
+				(font
+					(size 1.27 1.27)
+				)
+				(hide yes)
+			)
+		)
+		(property "Description" "Generic connector, single row, 01x03, script generated"
+			(at 210.82 110.49 0)
+			(effects
+				(font
+					(size 1.27 1.27)
+				)
+				(hide yes)
+			)
+		)
+		(property "Sim.Type" ""
+			(at 210.82 110.49 0)
+			(effects
+				(font
+					(size 1.27 1.27)
+				)
+				(hide yes)
+			)
+		)
+		(pin "3"
+		)
+		(pin "2"
+		)
+		(pin "1"
+		)
+		(instances
+			(project "BRS_HW_v1"
+				(path "/aaddc341-7c9c-4d67-a2d2-1ee9911ff161/6d2925c6-6c14-408e-a8be-7c6147054c34"
+					(reference "J10")
+					(unit 1)
+				)
+			)
+		)
+	)
+	(symbol
 		(lib_id "Device:C_Small")
 		(at 193.04 53.34 0)
@@
 					(unit 1)
 				)
+			)
+		)
+	)
+	(symbol
+		(lib_id "power:VCC")
+		(at 204.47 106.68 0)
+		(unit 1)
+		(exclude_from_sim no)
+		(in_bom yes)
+		(on_board yes)
+		(dnp no)
+		(fields_autoplaced yes)
+		(property "Reference" "#PWR097"
+			(at 204.47 110.49 0)
+			(effects
+				(font
+					(size 1.27 1.27)
+				)
+				(hide yes)
+			)
+		)
+		(property "Value" "VCC"
+			(at 204.47 101.6 0)
+			(effects
+				(font
+					(size 1.27 1.27)
+				)
+			)
+		)
+		(property "Footprint" ""
+			(at 204.47 106.68 0)
+			(effects
+				(font
+					(size 1.27 1.27)
+				)
+				(hide yes)
+			)
+		)
+		(property "Datasheet" ""
+			(at 204.47 106.68 0)
+			(effects
+				(font
+					(size 1.27 1.27)
+				)
+				(hide yes)
+			)
+		)
+		(property "Description" "Power symbol creates a global label with name \"VCC\""
+			(at 204.47 106.68 0)
+			(effects
+				(font
+					(size 1.27 1.27)
+				)
+				(hide yes)
+			)
+		)
+		(pin "1"
+		)
+		(instances
+			(project "BRS_HW_v1"
+				(path "/aaddc341-7c9c-4d67-a2d2-1ee9911ff161/6d2925c6-6c14-408e-a8be-7c6147054c34"
+					(reference "#PWR097")
+					(unit 1)
+				)

Commit message: Working on power source
Parts:
- removed D1, D2: TBD, Diode_SMD:D_SOD-123, symbol Device:D_Schottky_Small
- removed Q1: PMOS, Package_TO_SOT_SMD:SOT-23, symbol Simulation_SPICE:PMOS
- added C33, C34: 10u, Capacitor_SMD:C_0402_1005Metric, symbol Device:C_Small
- added C35, C36, C37: 100n, Capacitor_SMD:C_0402_1005Metric, symbol Device:C_Small
- added C38: 100u, Capacitor_SMD:C_0402_1005Metric, symbol Device:C_Small
- added J11: BACKUP_BAT, Connector_Molex:Molex_Micro-Fit_3.0_43045-0412_2x02_P3.00mm_Vertical, symbol Connector_Generic:Conn_02x02_Odd_Even
- added JP1, JP12: USB_PWR_JP, Jumper:SolderJumper-2_P1.3mm_Open_RoundedPad1.0x1.5mm, symbol Jumper:Jumper_2_Small_Open
- added Q1, Q9: AO3401A, Package_TO_SOT_SMD:SOT-23, symbol Transistor_FET:AO3401A
- added R35: 1k, Resistor_SMD:R_0402_1005Metric, symbol Device:R_Small
- added R36: 2k, Resistor_SMD:R_0402_1005Metric, symbol Device:R_Small
- added R37, R38: 62k, Resistor_SMD:R_0402_1005Metric, symbol Device:R_Small
- added R39, R42: 1M, Resistor_SMD:R_0402_1005Metric, symbol Device:R_Small
- added R40: 270k, Resistor_SMD:R_0402_1005Metric, symbol Device:R_Small
- added R41: 56k, Resistor_SMD:R_0402_1005Metric, symbol Device:R_Small
- added R43, R44: 150k, Resistor_SMD:R_0402_1005Metric, symbol Device:R_Small
- added R45: 100k, Resistor_SMD:R_0402_1005Metric, symbol Device:R_Small
- added R46, R? (x2): 10k, Resistor_SMD:R_0402_1005Metric, symbol Device:R_Small
- added TP2, TP3: TestPoint_Small, TestPoint:TestPoint_Pad_D1.5mm, symbol Connector:TestPoint_Small
- added U9: TPS2121, BRS_Footprints:VQFN-HR, symbol BRS_Library:TPS2121
- C1, C2, C3, C4, C5: footprint Capacitor_SMD:C_0603_1608Metric -> Capacitor_SMD:C_0402_1005Metric
- J1: value BATTERY -> MAIN_BAT
- JP2: footprint BRS_Footprints:SMD_SolderJumper_Small -> BRS_Footprints:SMD_SolderJumper_Micro
- R1: footprint Resistor_SMD:R_0603_1608Metric -> Resistor_SMD:R_0402_1005Metric
- renumbered JP1 to JP13
Connections:
- net BAT+ is gone; now on net M_BAT+: J1.1 (Pin_1), J1.3 (Pin_3)
- net GND: now also C33.2, C34.2, C35.2, C36.2, C37.2, C38.2, J11.2 (Pin_2), J11.4 (Pin_4), R35.2, R36.2, R41.2, R45.2, R46.2, R?.2, R?.2, U9.12 (GND), U9.9 (ST)
- net HV_PWR_IN: now also C38.1
- net VBUS: now also Q9.2 (S), TP3.1
- net M_BAT+: now reaches TP1.1
- net M_BAT+: now also C33.1, C35.1, JP1.1 (A)
- net at JP13.1 (A): now also Q9.3 (D)
- net +BATT: no longer names the net of SW1.1, SW1.2, SW1.3
- net +BATT: now also U9.1 (OUT), U9.8 (OUT); no longer JP13.2 (B)
- new net: R37.1, R39.2, U9.5 (OV1)
- new net: R35.1, R37.2
- new net: R43.2, R45.1, U9.3 (CP2)
- new net: R44.2, R46.1
- new net: R41.1, U9.10 (ILIM)
- new net: C37.1, U9.11 (SS)
- new net: R38.1, R40.2, U9.4 (OV2)
- new net: R42.2, R44.1, U9.6 (PR1)
- new net: Q1.1 (G), R?.1
- new net: JP12.1 (A), Q1.3 (D)
- new net: R36.1, R38.2
- new net: Q9.1 (G), R?.1
- new net B_BAT+: C34.1, C36.1, J11.1 (Pin_1), J11.3 (Pin_3), Q1.2 (S), TP2.1
- new net PWR_IN1: JP1.2 (B), R39.1, R42.1, U9.7 (IN1)
- new net PWR_IN2: JP12.2 (B), JP13.2 (B), R40.1, R43.1, U9.2 (IN2)
- no-connect marks 4 -> 3
Other:
- note added: "**TPS2121 design** ○ Requirements: • V_{IN1} = 14.8V nominal, within range 16.8V ~ 12.0V (4-cell LiPo) • V_{IN2} = 3.7V nominal, within range 5.0V ~ 3.0V (USB or backup LiPo) • I_{OUT_{(max)}} = 2A • C_{L} = 100uF • I_{INRUSH} = 100mA Note: USB will be used for debugging only, so calculations will consider backup LiPo voltage in IN2. ○ XCOMP mode: • If V_{CP2} ≤ V_{PR1} => VOUT = IN1 • If V_{CP2}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"
- moved on the sheet: C1, C2, C3, C4, C5, D3, J1, J10, J2, J8, J9, JP13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
