File: Hardware/Storage.kicad_sch (KiCad schematic)
At the start: 0 parts

Commit message: Developing HW
Parts:
- added C28: 10uF, Capacitor_SMD:C_0603_1608Metric, symbol Device:C_Small
- added C29: 100nF, Capacitor_SMD:C_0603_1608Metric, symbol Device:C_Small
- added J7: Micro_SD_Card, symbol Connector:Micro_SD_Card
- added Q7, Q8: AO3401A, Package_TO_SOT_SMD:SOT-23, symbol Transistor_FET:AO3401A
- added R28, R29: 10k, symbol Device:R_Small
- added U3: CAT811TTBI-GT3, Package_TO_SOT_SMD:SOT-143, symbol Power_Supervisor:CAT811TTBI-GT3
Connections:
- new net: Q8.1 (G), R29.1, U3.2 (~{RESET})
- new net: Q7.1 (G), Q8.2 (S), R28.2
- new net GND: C28.2, C29.2, J7.6 (VSS), R28.1, U3.1 (GND)
- new net SD_PWR: C28.1, C29.1, J7.4 (VDD), Q7.2 (S)
- new net SPI_MISO: J7.7 (DAT0)
- new net SPI_MOSI: J7.3 (CMD)
- new net SPI_SCK: J7.5 (CLK)
- new net SPI_SS1: J7.2 (DAT3/CD)
- new net VCC: Q7.3 (D), Q8.3 (D), R29.2, U3.4 (VCC)
- no-connect marks 0 -> 4

Commit message: Developing HW
Parts:
- added C22: 10uF, Capacitor_SMD:C_0603_1608Metric, symbol Device:C_Small
- added C23: 100nF, Capacitor_SMD:C_0603_1608Metric, symbol Device:C_Small
- added C24: 10nF, Capacitor_SMD:C_0603_1608Metric, symbol Device:C_Small
- added JP5: WP_JP, Jumper:SolderJumper-2_P1.3mm_Open_RoundedPad1.0x1.5mm, symbol Jumper:Jumper_2_Small_Open
- added R13: 100k, Resistor_SMD:R_0603_1608Metric, symbol Device:R_Small
- added R14, R15: 51k, Resistor_SMD:R_0603_1608Metric, symbol Device:R_Small
- added U5: W25Q128JVS, Package_SO:SOIC-8_5.23x5.23mm_P1.27mm, symbol Memory_Flash:W25Q128JVS
- J5: renamed from J7; footprint (none) -> Connector_Card:microSD_HC_Wuerth_693072010801
- R11: renamed from R29; footprint (none) -> Resistor_SMD:R_0603_1608Metric
- R12: renamed from R28; footprint (none) -> Resistor_SMD:R_0603_1608Metric
- renumbered C28 to C20, C29 to C21, Q8 to Q3, Q7 to Q4, U3 to U4
Connections:
- net GND: now also C22.2, C23.2, C24.2, JP5.1 (A), U5.4 (GND)
- net VCC: now also R13.2, R14.2, R15.2
- net SD_PWR renamed STRG_PWR
- net STRG_PWR: now also C22.1, C23.1, U5.8 (VCC)
- net SPI_MISO renamed SPI2_MISO
- net SPI2_MISO: now also U5.2 (DO(IO1))
- net SPI_MOSI renamed SPI2_MOSI
- net SPI2_MOSI: now also U5.5 (DI(IO0))
- net SPI_SCK renamed SPI2_SCK
- net SPI2_SCK: now also U5.6 (CLK)
- net SPI_SS1 renamed SPI2_NSS1
- net SPI2_NSS1: now also R15.1
- new net: C24.1, JP5.2 (B), R13.1, U5.3 (IO2)
- new net SPI2_NSS0: R14.1, U5.1 (~{CS})
- no-connect marks 4 -> 5
Other:
- note added: "IO2: /WP IO3: /HOLD or /RESET"
- moved on the sheet: C20, C21, J5, Q3, Q4, R11, R12, U4

Commit message: Developing HW - routing
Parts:
- JP5: footprint Jumper:SolderJumper-2_P1.3mm_Open_RoundedPad1.0x1.5mm -> Connector_PinHeader_2.54mm:PinHeader_1x02_P2.54mm_Vertical
Changed lines of the file:
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@@
 			)
 		)
-		(property "Footprint" "Jumper:SolderJumper-2_P1.3mm_Open_RoundedPad1.0x1.5mm"
+		(property "Footprint" "Connector_PinHeader_2.54mm:PinHeader_1x02_P2.54mm_Vertical"
 			(at 153.67 119.38 0)
 			(effects

Commit message: Working on power source
Parts:
- C20, C21, C22, C23, C24: footprint Capacitor_SMD:C_0603_1608Metric -> Capacitor_SMD:C_0402_1005Metric
- R11, R12, R13, R14, R15: footprint Resistor_SMD:R_0603_1608Metric -> Resistor_SMD:R_0402_1005Metric
Changed lines of the file:
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@@
 			)
 		)
-		(property "Footprint" "Capacitor_SMD:C_0603_1608Metric"
+		(property "Footprint" "Capacitor_SMD:C_0402_1005Metric"
 			(at 210.82 106.68 0)
 			(effects
@@
 			)
 		)
-		(property "Footprint" "Resistor_SMD:R_0603_1608Metric"
+		(property "Footprint" "Resistor_SMD:R_0402_1005Metric"
 			(at 158.75 115.57 0)
 			(effects
@@
 			)
 		)
-		(property "Footprint" "Resistor_SMD:R_0603_1608Metric"
+		(property "Footprint" "Resistor_SMD:R_0402_1005Metric"
 			(at 81.28 125.73 0)
 			(effects
@@
 			)
 		)
-		(property "Footprint" "Capacitor_SMD:C_0603_1608Metric"
+		(property "Footprint" "Capacitor_SMD:C_0402_1005Metric"
 			(at 158.75 123.19 0)
 			(effects
@@
 			)
 		)
-		(property "Footprint" "Resistor_SMD:R_0603_1608Metric"
+		(property "Footprint" "Resistor_SMD:R_0402_1005Metric"
 			(at 81.28 118.11 0)
 			(effects
@@
 			)
 		)
-		(property "Footprint" "Capacitor_SMD:C_0603_1608Metric"
+		(property "Footprint" "Capacitor_SMD:C_0402_1005Metric"
 			(at 147.32 57.15 0)
 			(effects
@@
 			)
 		)
-		(property "Footprint" "Capacitor_SMD:C_0603_1608Metric"
+		(property "Footprint" "Capacitor_SMD:C_0402_1005Metric"
 			(at 215.9 106.68 0)
 			(effects
@@
 			)
 		)
-		(property "Footprint" "Resistor_SMD:R_0603_1608Metric"
+		(property "Footprint" "Resistor_SMD:R_0402_1005Metric"
 			(at 76.2 62.23 0)
 			(effects
@@
 			)
 		)
-		(property "Footprint" "Resistor_SMD:R_0603_1608Metric"
+		(property "Footprint" "Resistor_SMD:R_0402_1005Metric"
 			(at 67.31 46.99 0)
 			(effects
@@
 			)
 		)
-		(property "Footprint" "Capacitor_SMD:C_0603_1608Metric"
+		(property "Footprint" "Capacitor_SMD:C_0402_1005Metric"
 			(at 142.24 57.15 0)
 			(effects
